Commit message: pi15 vel pen

File: my_pybullet_envs/assets/laikago/laikago_toes_limits.urdf (robot description, URDF)
Before this commit: robot plane, 17 links, 16 joints
Links:
- link FL_lower_leg: geometry collision mesh filename=lower_leg_3.stl scale=1 1 1; visual mesh filename=lower_leg3.obj scale=1 1 1
- link FR_lower_leg: geometry collision mesh filename=lower_leg_3.stl scale=1 1 1; visual mesh filename=lower_leg3.obj scale=1 1 1
- link RL_lower_leg: geometry collision mesh filename=lower_leg_3.stl scale=1 1 1; visual mesh filename=lower_leg3.obj scale=1 1 1
- link RR_lower_leg: geometry collision mesh filename=lower_leg_3.stl scale=1 1 1; visual mesh filename=lower_leg3.obj scale=1 1 1
